Commit message: mujoco is a bit scuffed

File: drawings/Triped_description/urdf/Triped.xacro (robot description, xacro)
@@ -2,9 +2,15 @@
 <robot name="Triped" xmlns:xacro="http://www.ros.org/wiki/xacro">
 <mujoco>
-  <compiler meshdir="../meshes/" balanceinertia="true" />
+  <compiler meshdir="../meshes/" balanceinertia="true" discardvisual="false" />
 </mujoco>
 <xacro:include filename="$(find Triped_description)/urdf/materials.xacro" />
 <xacro:include filename="$(find Triped_description)/urdf/Triped.trans" />
 <xacro:include filename="$(find Triped_description)/urdf/Triped.gazebo" />
+<link name="world"/>
+<joint name="floating_base" type="floating">
+  <origin rpy="0 0 0" xyz="0 0 0"/>
+  <parent link="world"/>
+  <child link="base_link"/>
+</joint>
 <link name="base_link">
   <inertial>

Commit message: tested simplification

File: drawings/Triped_description/urdf/Triped.xacro (robot description, xacro)
@@ -7,10 +7,10 @@
 <xacro:include filename="$(find Triped_description)/urdf/Triped.trans" />
 <xacro:include filename="$(find Triped_description)/urdf/Triped.gazebo" />
-<link name="world"/>
+<!-- <link name="world"/>
 <joint name="floating_base" type="floating">
   <origin rpy="0 0 0" xyz="0 0 0"/>
   <parent link="world"/>
   <child link="base_link"/>
-</joint>
+</joint> -->
 <link name="base_link">
   <inertial>
@@ -26,10 +26,10 @@
     <material name="silver"/>
   </visual>
-  <collision>
+  <!-- <collision>
     <origin xyz="0 0 0" rpy="0 0 0"/>
     <geometry>
       <mesh filename="package://Triped_description/meshes/base_link.stl" scale="0.001 0.001 0.001"/>
     </geometry>
-  </collision>
+  </collision> -->
 </link>
 <link name="servo_7_1">
@@ -46,10 +46,10 @@
     <material name="silver"/>
   </visual>
-  <collision>
+  <!-- <collision>
     <origin xyz="0.334457 -0.013741 0.052031" rpy="0 0 0"/>
     <geometry>
       <mesh filename="package://Triped_description/meshes/servo_7_1.stl" scale="0.001 0.001 0.001"/>
     </geometry>
-  </collision>
+  </collision> -->
 </link>
 <link name="servo_8_1">
@@ -66,10 +66,10 @@
     <material name="silver"/>
   </visual>
-  <collision>
+  <!-- <collision>
     <origin xyz="0.29223 0.032482 0.052031" rpy="0 0 0"/>
     <geometry>
       <mesh filename="package://Triped_description/meshes/servo_8_1.stl" scale="0.001 0.001 0.001"/>
     </geometry>
-  </collision>
+  </collision> -->
 </link>
 <link name="servo_9_1">
@@ -86,10 +86,10 @@
     <material name="silver"/>
   </visual>
-  <collision>
+  <!-- <collision>
     <origin xyz="0.273313 -0.027199 0.052031" rpy="0 0 0"/>
     <geometry>
       <mesh filename="package://Triped_description/meshes/servo_9_1.stl" scale="0.001 0.001 0.001"/>
     </geometry>
-  </collision>
+  </collision> -->
 </link>
 <link name="servo_6_1">
@@ -106,10 +106,10 @@
     <material name="silver"/>
   </visual>
-  <collision>
+  <!-- <collision>
     <origin xyz="0.269334 -0.024591 0.021891" rpy="0 0 0"/>
     <geometry>
       <mesh filename="package://Triped_description/meshes/servo_6_1.stl" scale="0.001 0.001 0.001"/>
     </geometry>
-  </collision>
+  </collision> -->
 </link>
 <link name="servo_5_1">
@@ -126,10 +126,10 @@
     <material name="silver"/>
   </visual>
-  <collision>
+  <!-- <collision>
     <origin xyz="0.296478 0.034624 0.021891" rpy="0 0 0"/>
     <geometry>
       <mesh filename="package://Triped_description/meshes/servo_5_1.stl" scale="0.001 0.001 0.001"/>
     </geometry>
-  </collision>
+  </collision> -->
 </link>
 <link name="servo_4_1">
@@ -146,10 +146,10 @@
     <material name="silver"/>
   </visual>
-  <collision>
+  <!-- <collision>
     <origin xyz="0.334188 -0.01849 0.021891" rpy="0 0 0"/>
     <geometry>
       <mesh filename="package://Triped_description/meshes/servo_4_1.stl" scale="0.001 0.001 0.001"/>
     </geometry>
-  </collision>
+  </collision> -->
 </link>
 <link name="servo_3_1">
@@ -166,10 +166,10 @@
     <material name="silver"/>
   </visual>
-  <collision>
+  <!-- <collision>
     <origin xyz="0.297718 -0.04981 0.016881" rpy="0 0 0"/>
     <geometry>
       <mesh filename="package://Triped_description/meshes/servo_3_1.stl" scale="0.001 0.001 0.001"/>
     </geometry>
-  </collision>
+  </collision> -->
 </link>
 <link name="servo_2_1">
@@ -186,10 +186,10 @@
     <material name="silver"/>
   </visual>
-  <collision>
+  <!-- <collision>
     <origin xyz="0.260446 0.022652 0.016881" rpy="0 0 0"/>
     <geometry>
       <mesh filename="package://Triped_description/meshes/servo_2_1.stl" scale="0.001 0.001 0.001"/>
     </geometry>
-  </collision>
+  </collision> -->
 </link>
 <link name="servo_1_1">
@@ -206,10 +206,10 @@
     <material name="silver"/>
   </visual>
-  <collision>
+  <!-- <collision>
     <origin xyz="0.341836 0.0187 0.016881" rpy="0 0 0"/>
     <geometry>
       <mesh filename="package://Triped_description/meshes/servo_1_1.stl" scale="0.001 0.001 0.001"/>
     </geometry>
-  </collision>
+  </collision> -->
 </link>
 <link name="holder_3_1">
@@ -226,10 +226,10 @@
     <material name="silver"/>
   </visual>
-  <collision>
+  <!-- <collision>
     <origin xyz="0.254578 -0.03075 0.016881" rpy="0 0 0"/>
     <geometry>
       <mesh filename="package://Triped_description/meshes/holder_3_1.stl" scale="0.001 0.001 0.001"/>
     </geometry>
-  </collision>
+  </collision> -->
 </link>
 <link name="holder_2_1">
@@ -246,10 +246,10 @@
     <material name="silver"/>
   </visual>
-  <collision>
+  <!-- <collision>
     <origin xyz="0.298523 0.050483 0.016881" rpy="0 0 0"/>
     <geometry>
       <mesh filename="package://Triped_description/meshes/holder_2_1.stl" scale="0.001 0.001 0.001"/>
     </geometry>
-  </collision>
+  </collision> -->
 </link>
 <link name="holder_1_1">
@@ -266,10 +266,10 @@
     <material name="silver"/>
   </visual>
-  <collision>
+  <!-- <collision>
     <origin xyz="0.346899 -0.028191 0.016881" rpy="0 0 0"/>
     <geometry>
       <mesh filename="package://Triped_description/meshes/holder_1_1.stl" scale="0.001 0.001 0.001"/>
     </geometry>
-  </collision>
+  </collision> -->
 </link>
 <link name="leg_3_1">
@@ -286,10 +286,10 @@
     <material name="silver"/>
   </visual>
-  <collision>
+  <!-- <collision>
     <origin xyz="0.271097 -0.021567 0.016881" rpy="0 0 0"/>
     <geometry>
       <mesh filename="package://Triped_description/meshes/leg_3_1.stl" scale="0.001 0.001 0.001"/>
     </geometry>
-  </collision>
+  </collision> -->
 </link>
 <link name="leg_2_1">
@@ -306,10 +306,10 @@
     <material name="silver"/>
   </visual>
-  <collision>
+  <!-- <collision>
     <origin xyz="0.298216 0.031586 0.016881" rpy="0 0 0"/>
     <geometry>
       <mesh filename="package://Triped_description/meshes/leg_2_1.stl" scale="0.001 0.001 0.001"/>
     </geometry>
-  </collision>
+  </collision> -->
 </link>
 <link name="leg_1_1">
@@ -326,10 +326,10 @@
     <material name="silver"/>
   </visual>
-  <collision>
+  <!-- <collision>
     <origin xyz="0.330688 -0.018476 0.016881" rpy="0 0 0"/>
     <geometry>
       <mesh filename="package://Triped_description/meshes/leg_1_1.stl" scale="0.001 0.001 0.001"/>
     </geometry>
-  </collision>
+  </collision> -->
 </link>
 <link name="foot_3_1">
